File: BLR8812AF1 baseboard.kicad_pcb (KiCad board)
At the start: 2 copper layers, 38 x 38 mm, 29 parts, among them Q1 AO3401A, U1 BL-R8812AF1, U2 USBLC6-2SC6, U3 TPS82130, X1 TYPE-C-31-M-12

Commit message: Fixed PCB and gerber files
Routing:
- net /Vin: track 8.87 -> 6.71 mm
Changed lines of the file:
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@@
 	)
 	(segment
-		(start 71.347 37.415)
-		(end 69.4928 35.5608)
+		(start 70.6104 36.5768)
+		(end 70.6104 34.7734)
 		(width 1.2)
 		(layer "B.Cu")
@@
 	)
 	(segment
-		(start 71.347 38.431)
-		(end 71.347 37.415)
+		(start 69.4928 33.6558)
+		(end 69.4928 30.3284)
 		(width 1.2)
 		(layer "B.Cu")
@@
 	)
 	(segment
-		(start 69.4928 35.5608)
-		(end 69.4928 30.3284)
+		(start 70.6104 34.7734)
+		(end 69.4928 33.6558)
 		(width 1.2)
 		(layer "B.Cu")
